Commit message: des

File: velatrix_description/urdf/base/base.xacro (robot description, xacro)
@@ -5,15 +5,15 @@
     <inertial>
       <origin
-        xyz="0.00042875 -0.061971 0.081713"
+        xyz="0.00054048 -0.062075 0.083117"
         rpy="0 0 0" />
       <mass
         value="1.3113" />
       <inertia
-        ixx="0.0033177"
-        ixy="4.9122E-06"
-        ixz="7.4028E-06"
-        iyy="0.003064"
-        iyz="-8.1926E-08"
-        izz="0.0054243" />
+        ixx="0.0033172"
+        ixy="4.7101E-06"
+        ixz="-3.0227E-06"
+        iyy="0.0030647"
+        iyz="9.5934E-06"
+        izz="0.005424" />
     </inertial>
     <visual>
@@ -47,5 +47,5 @@
       link="base_link" />
     <origin
-      xyz="0 0 0"
+      xyz="0 0 0.0528"
       rpy="0 0 0" />
   </joint>

File: velatrix_description/urdf/drone/drone.xacro (robot description, xacro)
@@ -5,14 +5,14 @@
     <inertial>
       <origin
-        xyz="0.00067846 -0.00067196 0.007248"
-        rpy="0 0 0" />
-      <mass
-        value="0.0032755" />
+        xyz="0.00067968 -0.00067076 0.0072481"
+        rpy="0 0 0" />
+      <mass
+        value="0.0032756" />
       <inertia
         ixx="1.0525E-06"
-        ixy="3.2951E-12"
-        ixz="1.3765E-11"
+        ixy="1.4878E-11"
+        ixz="1.4188E-11"
         iyy="1.0524E-06"
-        iyz="-4.1733E-12"
+        iyz="-4.5597E-12"
         izz="2.081E-06" />
     </inertial>
@@ -45,6 +45,6 @@
     type="continuous">
     <origin
-      xyz="0.22783 -0.21833 0.066876"
-      rpy="-0.047092 -0.027781 -0.75024" />
+      xyz="0.22886 -0.21928 0.074949"
+      rpy="-0.047092 -0.070937 -0.75024" />
     <parent
       link="base_link" />
@@ -53,9 +53,4 @@
     <axis
       xyz="0 0 1" />
-    <limit
-      lower="0"
-      upper="0"
-      effort="0"
-      velocity="0" />
   </joint>
   <link
@@ -63,5 +58,5 @@
     <inertial>
       <origin
-        xyz="0.00095032 8.8059E-05 0.0072482"
+        xyz="0.00095025 8.8109E-05 0.0072482"
         rpy="0 0 0" />
       <mass
@@ -69,8 +64,8 @@
       <inertia
         ixx="1.0524E-06"
-        ixy="-2.9734E-11"
-        ixz="2.4635E-11"
+        ixy="-2.3008E-11"
+        ixz="2.4323E-11"
         iyy="1.0524E-06"
-        iyz="-7.8753E-12"
+        iyz="-7.6481E-12"
         izz="2.0809E-06" />
     </inertial>
@@ -111,9 +106,4 @@
     <axis
       xyz="0 0 1" />
-    <limit
-      lower="0"
-      upper="0"
-      effort="0"
-      velocity="0" />
   </joint>
   <link
@@ -168,10 +158,10 @@
       link="duct1" />
     <axis
-      xyz="0 0.10601 0.99436" />
+      xyz="0 0 1" />
     <limit
       lower="0"
       upper="1.571"
       effort="0.98"
-      velocity="1" />
+      velocity="1.0" />
   </joint>
   <link
@@ -227,9 +217,4 @@
     <axis
       xyz="0 0 1" />
-    <limit
-      lower="0"
-      upper="0"
-      effort="0"
-      velocity="1" />
   </joint>
   <link
@@ -284,10 +269,10 @@
       link="duct2" />
     <axis
-      xyz="0 0.022049 0.99976" />
+      xyz="0 0 1" />
     <limit
       lower="0"
       upper="1.571"
       effort="0.98"
-      velocity="1" />
+      velocity="1.0" />
   </joint>
   <link
@@ -343,9 +328,4 @@
     <axis
       xyz="0 0 1" />
-    <limit
-      lower="0"
-      upper="0"
-      effort="0"
-      velocity="0" />
   </joint>
 </robot>

File: velatrix_description/urdf/leg/leg_1.xacro (robot description, xacro)
@@ -1,9 +1,8 @@
 <?xml version="1.0"?>
 <robot xmlns:xacro="http://www.ros.org/wiki/xacro">
-<link
-    name="c1">
+  <link name="c1">
     <inertial>
       <origin
-        xyz="0.030616 -0.0027342 -0.023249"
+        xyz="0.030615 -0.0027342 -0.026849"
         rpy="0 0 0" />
       <mass
@@ -41,9 +40,7 @@
     </collision>
   </link>
-  <joint
-    name="c1_jt"
-    type="revolute">
+  <joint name="c1_jt" type="revolute">
     <origin
-      xyz="0.039287 0.06031 0.04925"
+      xyz="0.039287 0.06031 0.05285"
       rpy="0 -0.0002253 0.9751" />
     <parent
@@ -52,13 +49,12 @@
       link="c1" />
     <axis
-      xyz="-0.0002253 0 -1" />
+      xyz="0 0 1" />
     <limit
-      lower="0.785"
-      upper="2.356"
+      lower="-0.785"
+      upper="0.785"
       effort="2.4"
-      velocity="1" />
+      velocity="1.0" />
   </joint>
-  <link
-    name="f1">
+  <link name="f1">
     <inertial>
       <origin
@@ -99,9 +95,7 @@
     </collision>
   </link>
-  <joint
-    name="f1_jt"
-    type="revolute">
+  <joint name="f1_jt" type="revolute">
     <origin
-      xyz="0.054484 -0.027961 -0.013852"
+      xyz="0.054484 -0.027961 -0.017452"
       rpy="1.5708 0 0" />
     <parent
@@ -110,13 +104,12 @@
       link="f1" />
     <axis
-      xyz="0 0 -1" />
+      xyz="0 0 1" />
     <limit
-      lower="0.785"
-      upper="2.356"
+      lower="-0.785"
+      upper="0.785"
       effort="2.4"
-      velocity="1" />
+      velocity="1.0" />
   </joint>
-  <link
-    name="t1">
+  <link name="t1">
     <inertial>
       <origin
@@ -157,7 +150,5 @@
     </collision>
   </link>
-  <joint
-    name="t1_jt"
-    type="revolute">
+  <joint name="t1_jt" type="revolute">
     <origin
       xyz="0.06677 0.021017 -0.0457"
@@ -168,9 +159,9 @@
       link="t1" />
     <axis
-      xyz="0 0 -1" />
+      xyz="0 0 1" />
     <limit
-      lower="0.785"
-      upper="2.356"
-      effort="1"
+      lower="-0.785"
+      upper="0.785"
+      effort="1.0"
       velocity="2.4" />
   </joint>

File: velatrix_description/urdf/leg/leg_2.xacro (robot description, xacro)
@@ -5,5 +5,5 @@
     <inertial>
       <origin
-        xyz="0.030616 -0.0027342 -0.023249"
+        xyz="0.030615 -0.0027342 -0.026849"
         rpy="0 0 0" />
       <mass
@@ -45,5 +45,5 @@
     type="revolute">
     <origin
-      xyz="0.070023 -0.00036228 0.04925"
+      xyz="0.070023 -0.00036228 0.05285"
       rpy="0 -0.0002253 0.028762" />
     <parent
@@ -52,10 +52,10 @@
       link="c2" />
     <axis
-      xyz="-0.0002253 0 -1" />
+      xyz="0 0 1" />
     <limit
-      lower="0.785"
-      upper="2.356"
+      lower="-0.785"
+      upper="0.785"
       effort="2.4"
-      velocity="1" />
+      velocity="1.0" />
   </joint>
   <link
@@ -103,5 +103,5 @@
     type="revolute">
     <origin
-      xyz="0.054484 -0.027961 -0.013852"
+      xyz="0.054484 -0.027961 -0.017452"
       rpy="1.5708 0 0" />
     <parent
@@ -110,10 +110,10 @@
       link="f2" />
     <axis
-      xyz="0 0 -1" />
+      xyz="0 0 1" />
     <limit
-      lower="0.785"
-      upper="2.356"
+      lower="-0.785"
+      upper="0.785"
       effort="2.4"
-      velocity="1" />
+      velocity="1.0" />
   </joint>
   <link
@@ -168,10 +168,10 @@
       link="t2" />
     <axis
-      xyz="0 0 -1" />
+      xyz="0 0 1" />
     <limit
-      lower="0.785"
-      upper="2.356"
+      lower="-0.785"
+      upper="0.785"
       effort="2.4"
-      velocity="1" />
+      velocity="1.0" />
   </joint>
 </robot>

File: velatrix_description/urdf/leg/leg_3.xacro (robot description, xacro)
@@ -1,9 +1,9 @@
 <?xml version="1.0"?>
 <robot xmlns:xacro="http://www.ros.org/wiki/xacro">
- <link
+  <link
     name="c3">
     <inertial>
       <origin
-        xyz="0.030616 -0.0027342 -0.023249"
+        xyz="0.030615 -0.0027342 -0.026849"
         rpy="0 0 0" />
       <mass
@@ -45,5 +45,5 @@
     type="revolute">
     <origin
-      xyz="0.041807 -0.05834 0.04925"
+      xyz="0.041807 -0.05834 0.05285"
       rpy="0 -0.0002253 -0.92041" />
     <parent
@@ -52,10 +52,10 @@
       link="c3" />
     <axis
-      xyz="-0.0002253 0 -1" />
+      xyz="0 0 1" />
     <limit
-      lower="0.785"
-      upper="2.356"
+      lower="-0.785"
+      upper="0.785"
       effort="2.4"
-      velocity="1" />
+      velocity="1.0" />
   </joint>
   <link
@@ -103,5 +103,5 @@
     type="revolute">
     <origin
-      xyz="0.054484 -0.027961 -0.013852"
+      xyz="0.054484 -0.027961 -0.017452"
       rpy="1.5708 0 0" />
     <parent
@@ -110,10 +110,10 @@
       link="f3" />
     <axis
-      xyz="0 0 -1" />
+      xyz="0 0 1" />
     <limit
-      lower="0.785"
-      upper="2.356"
+      lower="-0.785"
+      upper="0.785"
       effort="2.4"
-      velocity="1" />
+      velocity="1.0" />
   </joint>
   <link
@@ -168,10 +168,10 @@
       link="t3" />
     <axis
-      xyz="0 0 -1" />
+      xyz="0 0 1" />
     <limit
-      lower="0.785"
-      upper="2.356"
+      lower="-0.785"
+      upper="0.785"
       effort="2.4"
-      velocity="1" />
+      velocity="1.0" />
   </joint>
 </robot>

File: velatrix_description/urdf/leg/leg_4.xacro (robot description, xacro)
@@ -1,9 +1,9 @@
 <?xml version="1.0"?>
 <robot xmlns:xacro="http://www.ros.org/wiki/xacro">
-<link
+  <link
     name="c4">
     <inertial>
       <origin
-        xyz="0.030615 0.0027403 -0.023254"
+        xyz="0.030614 0.0027403 -0.026854"
         rpy="0 0 0" />
       <mass
@@ -45,5 +45,5 @@
     type="revolute">
     <origin
-      xyz="-0.039241 -0.061034 0.04925"
+      xyz="-0.039241 -0.061034 0.05285"
       rpy="0 -0.0002253 -2.2067" />
     <parent
@@ -52,8 +52,8 @@
       link="c4" />
     <axis
-      xyz="-0.0002253 0 -1" />
+      xyz="0 0 1" />
     <limit
-      lower="0.785"
-      upper="2.356"
+      lower="-0.785"
+      upper="0.785"
       effort="2.4"
       velocity="1" />
@@ -103,5 +103,5 @@
     type="revolute">
     <origin
-      xyz="0.054481 0.027975 -0.013863"
+      xyz="0.05448 0.027975 -0.017463"
       rpy="-1.5708 0 0" />
     <parent
@@ -110,10 +110,10 @@
       link="f4" />
     <axis
-      xyz="0 0 -1" />
+      xyz="0 0 1" />
     <limit
-      lower="0.785"
-      upper="2.356"
+      lower="-0.785"
+      upper="0.785"
       effort="2.4"
-      velocity="1" />
+      velocity="1.0" />
   </joint>
   <link
@@ -168,10 +168,10 @@
       link="t4" />
     <axis
-      xyz="0 0 -1" />
+      xyz="0 0 1" />
     <limit
-      lower="0.785"
-      upper="2.356"
+      lower="-0.785"
+      upper="0.785"
       effort="2.4"
-      velocity="1" />
+      velocity="1.0" />
   </joint>
 </robot>

File: velatrix_description/urdf/leg/leg_5.xacro (robot description, xacro)
@@ -1,9 +1,9 @@
 <?xml version="1.0"?>
 <robot xmlns:xacro="http://www.ros.org/wiki/xacro">
-<link
+  <link
     name="c5">
     <inertial>
       <origin
-        xyz="0.030615 0.0027403 -0.023254"
+        xyz="0.030614 0.0027403 -0.026854"
         rpy="0 0 0" />
       <mass
@@ -45,5 +45,5 @@
     type="revolute">
     <origin
-      xyz="-0.069977 -0.00036228 0.04925"
+      xyz="-0.069977 -0.00036228 0.05285"
       rpy="0 -0.0002253 -3.1161" />
     <parent
@@ -52,10 +52,10 @@
       link="c5" />
     <axis
-      xyz="-0.0002253 0 -1" />
+      xyz="0 0 1" />
     <limit
-      lower="0.785"
-      upper="2.356"
+      lower="-0.785"
+      upper="0.785"
       effort="2.4"
-      velocity="1" />
+      velocity="1.0" />
   </joint>
   <link
@@ -103,5 +103,5 @@
     type="revolute">
     <origin
-      xyz="0.054481 0.027975 -0.013863"
+      xyz="0.05448 0.027975 -0.017463"
       rpy="-1.5708 0 0" />
     <parent
@@ -110,10 +110,10 @@
       link="f5" />
     <axis
-      xyz="0 0 -1" />
+      xyz="0 0 1" />
     <limit
-      lower="0.785"
-      upper="2.356"
+      lower="-0.785"
+      upper="0.785"
       effort="2.4"
-      velocity="1" />
+      velocity="1.0" />
   </joint>
   <link
@@ -168,10 +168,10 @@
       link="t5" />
     <axis
-      xyz="0 0 -1" />
+      xyz="0 0 1" />
     <limit
-      lower="0.785"
-      upper="2.356"
+      lower="-0.785"
+      upper="0.785"
       effort="2.4"
-      velocity="1" />
+      velocity="1.0" />
   </joint>
 </robot>

File: velatrix_description/urdf/leg/leg_6.xacro (robot description, xacro)
@@ -1,9 +1,9 @@
 <?xml version="1.0"?>
 <robot xmlns:xacro="http://www.ros.org/wiki/xacro">
- <link
+  <link
     name="c6">
     <inertial>
       <origin
-        xyz="0.030615 0.0027403 -0.023254"
+        xyz="0.030614 0.0027403 -0.026854"
         rpy="0 0 0" />
       <mass
@@ -45,5 +45,5 @@
     type="revolute">
     <origin
-      xyz="-0.038726 0.060651 0.04925"
+      xyz="-0.038726 0.060651 0.05285"
       rpy="0 -0.0002253 2.1693" />
     <parent
@@ -52,10 +52,10 @@
       link="c6" />
     <axis
-      xyz="-0.0002253 0 -1" />
+      xyz="0 0 1" />
     <limit
-      lower="0.785"
-      upper="2.356"
+      lower="-0.785"
+      upper="0.785"
       effort="2.4"
-      velocity="1" />
+      velocity="1.0" />
   </joint>
   <link
@@ -103,5 +103,5 @@
     type="revolute">
     <origin
-      xyz="0.054481 0.027975 -0.013863"
+      xyz="0.05448 0.027975 -0.017463"
       rpy="-1.5708 0 0" />
     <parent
@@ -110,10 +110,10 @@
       link="f6" />
     <axis
-      xyz="0 0 -1" />
+      xyz="0 0 1" />
     <limit
-      lower="0.785"
-      upper="2.356"
+      lower="-0.785"
+      upper="0.785"
       effort="2.4"
-      velocity="1" />
+      velocity="1.0" />
   </joint>
   <link
@@ -168,10 +168,10 @@
       link="t6" />
     <axis
-      xyz="0 0 -1" />
+      xyz="0 0 1" />
     <limit
-      lower="0.785"
-      upper="2.356"
+      lower="-0.785"
+      upper="0.785"
       effort="2.4"
-      velocity="1" />
+      velocity="1.0" />
   </joint>
 </robot>

File: velatrix_description/urdf/sensor/depth_camera.xacro (robot description, xacro)
@@ -1,19 +1,19 @@
 <?xml version="1.0"?>
 <robot xmlns:xacro="http://www.ros.org/wiki/xacro">
- <link
+  <link
     name="depth_camera">
     <inertial>
       <origin
-        xyz="0.00011447 -0.0038099 -0.001006"
+        xyz="5.7613E-05 -0.0034402 9.2747E-05"
         rpy="0 0 0" />
       <mass
-        value="0.0037619" />
+        value="0.0032848" />
       <inertia
-        ixx="2.9482E-07"
-        ixy="-4.5891E-10"
-        ixz="2.2255E-11"
-        iyy="6.1122E-07"
-        iyz="-1.2321E-10"
-        izz="3.21E-07" />
+        ixx="2.9286E-07"
+        ixy="-4.6644E-10"
+        ixz="2.1929E-11"
+        iyy="6.0022E-07"
+        iyz="-6.8969E-11"
+        izz="3.1133E-07" />
     </inertial>
     <visual>
@@ -28,5 +28,5 @@
         name="">
         <color
-          rgba="0.75294 0.75294 0.75294 1" />
+          rgba="0.37647 0.37647 0.37647 1" />
       </material>
     </visual>
@@ -51,6 +51,4 @@
     <child
       link="depth_camera" />
-    <axis
-      xyz="0 0 0" />
   </joint>
 </robot>

File: velatrix_description/urdf/sensor/lidar.xacro (robot description, xacro)
@@ -1,6 +1,5 @@
 <?xml version="1.0"?>
 <robot xmlns:xacro="http://www.ros.org/wiki/xacro">
-  <link
-    name="lidar">
+  <link name="lidar">
     <inertial>
       <origin
@@ -41,7 +40,5 @@
     </collision>
   </link>
-  <joint
-    name="lidar_jt"
-    type="fixed">
+  <joint name="lidar_jt" type="fixed">
     <origin
       xyz="2.3087E-05 -0.00036228 0.14781"
@@ -51,6 +48,4 @@
     <child
       link="lidar" />
-    <axis
-      xyz="0 0 0" />
   </joint>
 </robot>

File: velatrix_description/urdf/sensor/thermal_camera.xacro (robot description, xacro)
@@ -5,15 +5,15 @@
     <inertial>
       <origin
-        xyz="0.0022649 -0.0045666 -5.3595E-05"
+        xyz="0.0027024 -0.0044041 0.00040923"
         rpy="0 0 0" />
       <mass
-        value="0.0014693" />
+        value="0.0011581" />
       <inertia
-        ixx="7.6254E-08"
-        ixy="-8.9935E-13"
-        ixz="-2.2398E-11"
-        iyy="1.3203E-07"
-        iyz="7.6296E-14"
-        izz="5.7067E-08" />
+        ixx="7.427E-08"
+        ixy="-6.8145E-24"
+        ixz="-2.7603E-11"
+        iyy="1.2871E-07"
+        iyz="2.5154E-12"
+        izz="5.5021E-08" />
     </inertial>
     <visual>
@@ -28,5 +28,5 @@
         name="">
         <color
-          rgba="0.75294 0.75294 0.75294 1" />
+          rgba="0.79216 0.81961 0.93333 1" />
       </material>
     </visual>
@@ -45,5 +45,5 @@
     type="fixed">
     <origin
-      xyz="0.014989 0.13586 0.11642"
+      xyz="0.014989 0.13522 0.11643"
       rpy="-0.019827 0 0" />
     <parent
@@ -52,5 +52,5 @@
       link="thermal_camera" />
     <axis
-      xyz="1 0 0" />
+      xyz="0 0 0" />
   </joint>
 </robot>

File: velatrix_description/urdf/velatrix.urdf.xacro (robot description, xacro)
@@ -2,5 +2,5 @@
 <robot xmlns:xacro="http://www.ros.org/wiki/xacro" name="velatrix">
     <xacro:include filename="base/base.xacro"/>
-    <!-- <xacro:include filename="leg/leg_1.xacro"/>
+    <xacro:include filename="leg/leg_1.xacro"/>
     <xacro:include filename="leg/leg_2.xacro"/>
     <xacro:include filename="leg/leg_3.xacro"/>
@@ -8,4 +8,9 @@
     <xacro:include filename="leg/leg_5.xacro"/>
     <xacro:include filename="leg/leg_6.xacro"/>
- -->
+    <xacro:include filename="sensor/depth_camera.xacro"/>
+    <xacro:include filename="sensor/thermal_camera.xacro"/>
+    <xacro:include filename="sensor/lidar.xacro"/>
+    <xacro:include filename="drone/drone.xacro"/>
+    <xacro:include filename="gazebo.xacro"/>
+    <xacro:include filename="velatrix.ros2_control.xacro"/>
 </robot>
