Commit message: bot_colour_for_gazebo

File: velatrix_description/urdf/gazebo.xacro (robot description, xacro)
@@ -3,5 +3,11 @@
   <!-- Gazebo references for all links -->
   <gazebo reference="base_link">
-    <material>Gazebo/Grey</material>
+    <visual>
+      <material>
+        <ambient>1 0 0 1</ambient>
+        <diffuse>1 0 0 1</diffuse>
+        <specular>0.5 0.5 0.5 1</specular>
+      </material>
+    </visual>
     <mu1>0.8</mu1>
     <mu2>0.8</mu2>
@@ -10,5 +16,11 @@
   <!-- Leg 1 -->
   <gazebo reference="c1">
-    <material>Gazebo/Red</material>
+    <visual>
+      <material>
+        <ambient>0 0 0 1</ambient>
+        <diffuse>0 0 0 1</diffuse>
+        <specular>0.1 0.1 0.1 1</specular>
+      </material>
+    </visual>
     <mu1>0.8</mu1>
     <mu2>0.8</mu2>
@@ -16,5 +28,11 @@
   </gazebo>
   <gazebo reference="f1">
-    <material>Gazebo/DarkGrey</material>
+    <visual>
+      <material>
+        <ambient>1 0 0 1</ambient>
+        <diffuse>1 0 0 1</diffuse>
+        <specular>0.5 0.5 0.5 1</specular>
+      </material>
+    </visual>
     <mu1>0.8</mu1>
     <mu2>0.8</mu2>
@@ -22,5 +40,11 @@
   </gazebo>
   <gazebo reference="t1">
-    <material>Gazebo/Red</material>
+    <visual>
+      <material>
+        <ambient>0 0 0 1</ambient>
+        <diffuse>0 0 0 1</diffuse>
+        <specular>0.1 0.1 0.1 1</specular>
+      </material>
+    </visual>
     <mu1>1.0</mu1>
     <mu2>1.0</mu2>
@@ -31,5 +55,11 @@
   <!-- Leg 2 -->
   <gazebo reference="c2">
-    <material>Gazebo/Red</material>
+    <visual>
+      <material>
+        <ambient>0 0 0 1</ambient>
+        <diffuse>0 0 0 1</diffuse>
+        <specular>0.1 0.1 0.1 1</specular>
+      </material>
+    </visual>
     <mu1>0.8</mu1>
     <mu2>0.8</mu2>
@@ -37,5 +67,11 @@
   </gazebo>
   <gazebo reference="f2">
-    <material>Gazebo/Red</material>
+    <visual>
+      <material>
+        <ambient>1 0 0 1</ambient>
+        <diffuse>1 0 0 1</diffuse>
+        <specular>0.5 0.5 0.5 1</specular>
+      </material>
+    </visual>
     <mu1>0.8</mu1>
     <mu2>0.8</mu2>
@@ -43,5 +79,11 @@
   </gazebo>
   <gazebo reference="t2">
-    <material>Gazebo/Red</material>
+    <visual>
+      <material>
+        <ambient>0 0 0 1</ambient>
+        <diffuse>0 0 0 1</diffuse>
+        <specular>0.1 0.1 0.1 1</specular>
+      </material>
+    </visual>
     <mu1>1.0</mu1>
     <mu2>1.0</mu2>
@@ -52,5 +94,11 @@
   <!-- Leg 3 -->
   <gazebo reference="c3">
-    <material>Gazebo/Red</material>
+    <visual>
+      <material>
+        <ambient>0 0 0 1</ambient>
+        <diffuse>0 0 0 1</diffuse>
+        <specular>0.1 0.1 0.1 1</specular>
+      </material>
+    </visual>
     <mu1>0.8</mu1>
     <mu2>0.8</mu2>
@@ -58,5 +106,11 @@
   </gazebo>
   <gazebo reference="f3">
-    <material>Gazebo/Red</material>
+    <visual>
+      <material>
+        <ambient>1 0 0 1</ambient>
+        <diffuse>1 0 0 1</diffuse>
+        <specular>0.5 0.5 0.5 1</specular>
+      </material>
+    </visual>
     <mu1>0.8</mu1>
     <mu2>0.8</mu2>
@@ -64,5 +118,11 @@
   </gazebo>
   <gazebo reference="t3">
-    <material>Gazebo/Red</material>
+    <visual>
+      <material>
+        <ambient>0 0 0 1</ambient>
+        <diffuse>0 0 0 1</diffuse>
+        <specular>0.1 0.1 0.1 1</specular>
+      </material>
+    </visual>
     <mu1>1.0</mu1>
     <mu2>1.0</mu2>
@@ -73,5 +133,11 @@
   <!-- Leg 4 -->
   <gazebo reference="c4">
-    <material>Gazebo/Red</material>
+    <visual>
+      <material>
+        <ambient>0 0 0 1</ambient>
+        <diffuse>0 0 0 1</diffuse>
+        <specular>0.1 0.1 0.1 1</specular>
+      </material>
+    </visual>
     <mu1>0.8</mu1>
     <mu2>0.8</mu2>
@@ -79,5 +145,11 @@
   </gazebo>
   <gazebo reference="f4">
-    <material>Gazebo/Red</material>
+    <visual>
+      <material>
+        <ambient>1 0 0 1</ambient>
+        <diffuse>1 0 0 1</diffuse>
+        <specular>0.5 0.5 0.5 1</specular>
+      </material>
+    </visual>
     <mu1>0.8</mu1>
     <mu2>0.8</mu2>
@@ -85,5 +157,11 @@
   </gazebo>
   <gazebo reference="t4">
-    <material>Gazebo/Red</material>
+    <visual>
+      <material>
+        <ambient>0 0 0 1</ambient>
+        <diffuse>0 0 0 1</diffuse>
+        <specular>0.1 0.1 0.1 1</specular>
+      </material>
+    </visual>
     <mu1>1.0</mu1>
     <mu2>1.0</mu2>
@@ -94,5 +172,11 @@
   <!-- Leg 5 -->
   <gazebo reference="c5">
-    <material>Gazebo/Red</material>
+    <visual>
+      <material>
+        <ambient>0 0 0 1</ambient>
+        <diffuse>0 0 0 1</diffuse>
+        <specular>0.1 0.1 0.1 1</specular>
+      </material>
+    </visual>
     <mu1>0.8</mu1>
     <mu2>0.8</mu2>
@@ -100,5 +184,11 @@
   </gazebo>
   <gazebo reference="f5">
-    <material>Gazebo/Red</material>
+    <visual>
+      <material>
+        <ambient>1 0 0 1</ambient>
+        <diffuse>1 0 0 1</diffuse>
+        <specular>0.5 0.5 0.5 1</specular>
+      </material>
+    </visual>
     <mu1>0.8</mu1>
     <mu2>0.8</mu2>
@@ -106,5 +196,11 @@
   </gazebo>
   <gazebo reference="t5">
-    <material>Gazebo/Red</material>
+    <visual>
+      <material>
+        <ambient>0 0 0 1</ambient>
+        <diffuse>0 0 0 1</diffuse>
+        <specular>0.1 0.1 0.1 1</specular>
+      </material>
+    </visual>
     <mu1>1.0</mu1>
     <mu2>1.0</mu2>
@@ -115,5 +211,11 @@
   <!-- Leg 6 -->
   <gazebo reference="c6">
-    <material>Gazebo/Red</material>
+    <visual>
+      <material>
+        <ambient>0 0 0 1</ambient>
+        <diffuse>0 0 0 1</diffuse>
+        <specular>0.1 0.1 0.1 1</specular>
+      </material>
+    </visual>
     <mu1>0.8</mu1>
     <mu2>0.8</mu2>
@@ -121,5 +223,11 @@
   </gazebo>
   <gazebo reference="f6">
-    <material>Gazebo/Red</material>
+    <visual>
+      <material>
+        <ambient>1 0 0 1</ambient>
+        <diffuse>1 0 0 1</diffuse>
+        <specular>0.5 0.5 0.5 1</specular>
+      </material>
+    </visual>
     <mu1>0.8</mu1>
     <mu2>0.8</mu2>
@@ -127,5 +235,11 @@
   </gazebo>
   <gazebo reference="t6">
-    <material>Gazebo/Red</material>
+    <visual>
+      <material>
+        <ambient>0 0 0 1</ambient>
+        <diffuse>0 0 0 1</diffuse>
+        <specular>0.1 0.1 0.1 1</specular>
+      </material>
+    </visual>
     <mu1>1.0</mu1>
     <mu2>1.0</mu2>

File: velatrix_description/urdf/velatrix.ros2_control.xacro (robot description, xacro)
@@ -2,5 +2,4 @@
 <robot xmlns:xacro="http://www.ros.org/wiki/xacro">
   <xacro:macro name="velatrix_ros2_control" params="
-    name
     use_fake_hardware:=false
     fake_sensor_commands:=false
@@ -9,5 +8,4 @@
     initial_positions_file
     joint_limits_file
-    simulation_controllers
     ">
     <!-- Load configuration files -->
@@ -17,5 +15,5 @@
     <xacro:property name="initial_positions" value="${initial_positions_config}"/>
     <xacro:property name="joint_limits" value="${joint_limits_config['joint_limits']}"/>
-    <ros2_control name="${name}" type="system">
+    <ros2_control name="VelatrixSystem" type="system">
       <hardware>
         <xacro:if value="${sim_gazebo}">

File: velatrix_description/urdf/velatrix.urdf.xacro (robot description, xacro)
@@ -18,5 +18,4 @@
     <!-- ========== ROS2_CONTROL CONFIGURATION ========== -->
     <xacro:velatrix_ros2_control
-        name="VelatrixSystem"
         use_fake_hardware="$(arg use_fake_hardware)"
         fake_sensor_commands="$(arg fake_sensor_commands)"
@@ -25,11 +24,9 @@
         initial_positions_file="$(arg initial_positions_file)"
         joint_limits_file="$(arg joint_limits_file)"
-        simulation_controllers="$(arg simulation_controllers)"
     />
     <xacro:if value="$(arg sim_gazebo)">
         <gazebo>
-            <plugin filename="libign_ros2_control-system.so" name="ign_ros2_control::IgnitionROS2ControlPlugin">
-                <parameters>$(arg simulation_controllers)</parameters>
-                <controller_manager_node_name>controller_manager</controller_manager_node_name>
+            <plugin filename="gz_ros2_control-system" name="gz_ros2_control::GazeboSimROS2ControlPlugin">
+                <parameters>$(find velatrix_bringup)/config/hexapod_controller.yaml</parameters>
             </plugin>
         </gazebo>
@@ -37,8 +34,7 @@
     <xacro:if value="$(arg sim_ignition)">
         <gazebo>
-        <plugin filename="libign_ros2_control-system.so" name="ign_ros2_control::IgnitionROS2ControlPlugin">
-            <parameters>$(arg simulation_controllers)</parameters>
-            <controller_manager_node_name>controller_manager</controller_manager_node_name>
-        </plugin>
+            <plugin filename="gz_ros2_control-system" name="gz_ros2_control::GazeboSimROS2ControlPlugin">
+                <parameters>$(find velatrix_bringup)/config/hexapod_controller.yaml</parameters>
+            </plugin>
         </gazebo>
     </xacro:if>
